File: pcb/v0.1_eagle/OLM-env-sensor.sch (EAGLE design)
At the start: 10 parts, among them J1 1X2-3.5MM, U1 AM2302

Commit message: fixed wiring
Parts:
- removed JP3, JP4, JP5: M10", SparkFun-Connectors:M10"
- added C2: 1.0µ, resistor:C-EU025-024X044
- added IC1: LM358N, linear:LM358N
- added R2, R3, R4, R5: 10k, rcl:R-EU_0204/7
Connections:
- new net N$1: IC1A.-IN, IC1A.OUT, J1.1
- new net N$3: C2.1, IC1A.+IN, R2.1, R3.2
- new net N$6: IC1B.-IN, R4.2
- net 3.3V: no longer J1.1
- net AIO-0: now also IC1B.+IN, IC1B.OUT, R4.1; no longer JP3.4, JP4.4, JP5.4
- net DIO-0: no longer JP3.5, JP4.5, JP5.5
- net DIO-1: no longer JP3.6, JP4.6, JP5.6
- net DIO-2: no longer JP3.7, JP4.7, JP5.7
- net GND: now also C2.2, R3.1, R5.2; no longer JP3.2, JP4.2, JP5.2
- net MISO: no longer JP3.8, JP4.8, JP5.8
- net MOSI: no longer JP3.9, JP4.9, JP5.9
- net SCK: no longer JP3.10, JP4.10, JP5.10
- net VCC: no longer JP3.3, JP4.3, JP5.3
- net VIN: no longer JP3.1, JP4.1, JP5.1
Other:
- moved on the sheet: JP1
